File: artemis-board/charger_io.sch (KiCad schematic (older format))
At the start: 5 parts, among them J3 USB_B_Micro, J4 Solar in, U15 IP4220CZ6

Commit message: added comments, part numbers and extended marker
Parts:
- J3: Extended (none) -> Extended
- J4: value Solar in -> DC in; Extended (none) -> Extended
Changed lines of the file:
@@
 P 5600 3100
 F 0 "J4" H 5750 2800 50  0000 C CNN
-F 1 "Solar in" H 5700 2900 50  0000 C CNN
+F 1 "DC in" H 5700 2900 50  0000 C CNN
 F 2 "Connector_JST:JST_EH_S2B-EH_1x02_P2.50mm_Horizontal" H 5600 3100 50  0001 C CNN
 F 3 "https://datasheet.lcsc.com/szlcsc/1811051822_JST-Sales-America-S2B-XH-A-LF-SN_C157931.pdf" H 5600 3100 50  0001 C CNN
 F 4 "C225424" H 5600 3100 50  0001 C CNN "LCSC"
+F 5 "Extended" H 5600 3100 50  0001 C CNN "Extended"
 	1    5600 3100
 	-1   0    0    1
@@
 F 3 "https://datasheet.lcsc.com/szlcsc/1912111437_SHOU-HAN-MicroXNJ_C404969.pdf" H 3450 3150 50  0001 C CNN
 F 4 "C404969" H 3300 3200 50  0001 C CNN "LCSC"
+F 5 "Extended" H 3300 3200 50  0001 C CNN "Extended"
 	1    3300 3200
 	1    0    0    -1
